File: Hardware/kiCad_chessLab/power_board.kicad_sch (KiCad schematic)
At the start: 43 parts, among them IC1 MT3608, IC2 TP4056, IC3 DW01A-G, J1 DATA, J2 PWR, J3 AUX, Q1 FS8205A, Q2 AO3401A, SW1 SW_SPST, U1 BAT, U2 AMS1117-3.3

Commit message: NEW REFERENCES
Parts:
- Q1: footprint chessLab-footprints:SOP65P640X120-8N -> chessLab-footprints:SOT-23-6_L2.9-W1.6-P0.95-LS2.8-BR; symbol chessLab-symbols:FS8205A -> chessLab-symbols:FS8205A_C2830320
- U2: footprint Package_TO_SOT_SMD:SOT-223-3_TabPin2 -> chessLab-footprints:SOT-223-3_L6.5-W3.4-P2.30-LS7.0-BR; symbol Regulator_Linear:AMS1117-3.3 -> chessLab-symbols:AMS1117-3.3
Connections:
- net +3V3: no longer U2.2 (VO)
- net GND: no longer Q1.6 (S2_1), Q1.7 (S2_2), U2.1 (GND)
- net VSYS: no longer U2.3 (VI)
- net at C3.2, IC3.6 (GND), U1.1 (-_1)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: no longer Q1.2 (S1_1), Q1.3 (S1_2)
- net at IC3.1 (OD): no longer Q1.4 (G1)
- net at IC3.3 (OC): no longer Q1.5 (G2)
- net at Q1.1 (S1): no longer Q1.8 (D12_2)
Changed lines of the file:
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@@
 	)
 	(symbol
-		(lib_id "chessLab-symbols:FS8205A")
+		(lib_id "chessLab-symbols:FS8205A_C2830320")
 		(at 77.47 119.38 0)
 		(unit 1)
@@
 			)
 		)
-		(property "Footprint" "chessLab-footprints:SOP65P640X120-8N"
+		(property "Footprint" "chessLab-footprints:SOT-23-6_L2.9-W1.6-P0.95-LS2.8-BR"
 			(at 104.14 214.3 0)
 			(effects
@@
 	)
 	(symbol
-		(lib_id "Regulator_Linear:AMS1117-3.3")
+		(lib_id "chessLab-symbols:AMS1117-3.3")
 		(at 152.4 33.02 0)
 		(unit 1)
@@
 			)
 		)
-		(property "Footprint" "Package_TO_SOT_SMD:SOT-223-3_TabPin2"
+		(property "Footprint" "chessLab-footprints:SOT-223-3_L6.5-W3.4-P2.30-LS7.0-BR"
 			(at 152.4 27.94 0)
 			(effects
